Commit message: update .xacro file

File: my_robot/urdf/my_robot.xacro (robot description, xacro)
@@ -1,186 +1,188 @@
-<?xml version='1.0'?>
+<?xml version="1.0"?>
 <robot name="my_robot" xmlns:xacro="http://www.ros.org/wiki/xacro">
+  <xacro:include filename="$(find my_robot)/urdf/my_robot.gazebo" />
   <link name="robot_footprint"></link>
-  <xacro:include filename="$(find my_robot)/urdf/my_robot.gazebo" />
   <joint name="robot_footprint_joint" type="fixed">
     <origin xyz="0 0 0" rpy="0 0 0" />
-    <parent link="robot_footprint"/>
+    <parent link="robot_footprint" />
     <child link="chassis" />
   </joint>
-  <link name='chassis'>
+  <link name="chassis">
     <pose>0 0 0.1 0 0 0</pose>
     <inertial>
-      <mass value="15.0"/>
-      <origin xyz="0.0 0 0" rpy=" 0 0 0"/>
+      <mass value="15.0" />
+      <origin xyz="0 0 0" rpy="0 0 0" />
       <inertia
-          ixx="0.1" ixy="0" ixz="0"
-          iyy="0.1" iyz="0"
-          izz="0.1"
+        ixx="0.1" ixy="0" ixz="0"
+        iyy="0.1" iyz="0"
+        izz="0.1"
       />
     </inertial>
-    <collision name='collision'>
-      <origin xyz="0 0 0" rpy=" 0 0 0"/>
+    <collision name="chassis_collision_1">
+      <origin xyz="-.2 0 0" rpy="0 0 0" />
       <geometry>
-        <box size=".4 .2 .1"/>
+        <box size="1.0 .2 .1" />
       </geometry>
     </collision>
-    <visual name='chassis_visual'>
-      <origin xyz="0 0 0" rpy=" 0 0 0"/>
+    <visual name="chassis_visual_1">
+      <origin xyz="-.2 0 0" rpy="0 0 0" />
       <geometry>
-        <box size=".4 .2 .1"/>
+        <box size="1.0 .2 .1" />
       </geometry>
     </visual>
-    <collision name='back_caster_collision'>
-      <origin xyz="-0.15 0 -0.05" rpy=" 0 0 0"/>
+    <collision name="chassis_collision_2">
+      <origin xyz="0 0 0" rpy="0 0 0" />
       <geometry>
-        <sphere radius="0.0499"/>
+        <box size=".2 .6 .1" />
       </geometry>
     </collision>
-    <visual name='back_caster_visual'>
-      <origin xyz="-0.15 0 -0.05" rpy=" 0 0 0"/>
+    <visual name="chassis_visual_2">
+      <origin xyz="0 0 0" rpy="0 0 0" />
       <geometry>
-        <sphere radius="0.05"/>
+        <box size=".2 .6 .1" />
       </geometry>
     </visual>
-    <collision name='front_caster_collision'>
-      <origin xyz="0.15 0 -0.05" rpy=" 0 0 0"/>
+    <collision name="back_caster_collision">
+      <origin xyz="-0.65 0 -0.05" rpy="0 0 0" />
       <geometry>
-        <sphere radius="0.0499"/>
+        <sphere radius="0.0499" />
       </geometry>
     </collision>
-    <visual name='front_caster_visual'>
-      <origin xyz="0.15 0 -0.05" rpy=" 0 0 0"/>
+    <visual name="back_caster_visual">
+      <origin xyz="-0.65 0 -0.05" rpy="0 0 0" />
       <geometry>
-        <sphere radius="0.05"/>
+        <sphere radius="0.0499" />
+      </geometry>
+    </visual>
+    <collision name="front_caster_collision">
+      <origin xyz="0.25 0 -0.05" rpy="0 0 0" />
+      <geometry>
+        <sphere radius="0.0499" />
+      </geometry>
+    </collision>
+    <visual name="front_caster_visual">
+      <origin xyz="0.25 0 -0.05" rpy="0 0 0" />
+      <geometry>
+        <sphere radius="0.0499" />
       </geometry>
     </visual>
   </link>
-  <link name='left_wheel'>
-    <pose>0 0 0 0 0 0</pose>
+  <link name="left_wheel">
     <inertial>
-      <mass value="5.0"/>
-      <origin xyz="0.0 0 0" rpy=" 0 1.5707 1.5707"/>
+      <mass value="5.0" />
+      <origin xyz="0 0 0" rpy="0 1.5707 1.5707" />
       <inertia
-          ixx="0.1" ixy="0" ixz="0"
-          iyy="0.1" iyz="0"
-          izz="0.1"
+        ixx="0.1" ixy="0" ixz="0"
+        iyy="0.1" iyz="0"
+        izz="0.1"
       />
     </inertial>
-    <collision name='collision'>
-      <origin xyz="0 0 0" rpy=" 0 1.5707 1.5707"/>
+    <collision>
+      <origin xyz="0 0 0" rpy="0 1.5707 1.5707" />
       <geometry>
-        <cylinder radius="0.1" length="0.05"/>
+        <cylinder radius="0.1" length="0.05" />
       </geometry>
     </collision>
-    <visual name='left_wheel_visual'>
-      <origin xyz="0 0 0" rpy=" 0 1.5707 1.5707"/>
+    <visual>
+      <origin xyz="0 0 0" rpy="0 1.5707 1.5707" />
       <geometry>
-        <cylinder radius="0.1" length="0.05"/>
+        <cylinder radius="0.1" length="0.05" />
       </geometry>
     </visual>
   </link>
-  <link name='right_wheel'>
-    <pose>0 0 0 0 0 0</pose>
+  <link name="right_wheel">
     <inertial>
-      <mass value="5.0"/>
-      <origin xyz="0.0 0 0" rpy=" 0 1.5707 1.5707"/>
+      <mass value="5.0" />
+      <origin xyz="0 0 0" rpy="0 1.5707 1.5707" />
       <inertia
-          ixx="0.1" ixy="0" ixz="0"
-          iyy="0.1" iyz="0"
-          izz="0.1"
+        ixx="0.1" ixy="0" ixz="0"
+        iyy="0.1" iyz="0"
+        izz="0.1"
       />
     </inertial>
-    <collision name='collision'>
-      <origin xyz="0 0 0" rpy=" 0 1.5707 1.5707"/>
+    <collision>
+      <origin xyz="0 0 0" rpy="0 1.5707 1.5707" />
       <geometry>
-        <cylinder radius="0.1" length="0.05"/>
+        <cylinder radius="0.1" length="0.05" />
       </geometry>
     </collision>
-    <visual name='right_wheel_visual'>
-      <origin xyz="0 0 0" rpy=" 0 1.5707 1.5707"/>
+    <visual>
+      <origin xyz="0 0 0" rpy="0 1.5707 1.5707" />
       <geometry>
-        <cylinder radius="0.1" length="0.05"/>
+        <cylinder radius="0.1" length="0.05" />
       </geometry>
     </visual>
   </link>
+  <gazebo reference="left_wheel">
+    <material>Gazebo/Blue</material>
+  </gazebo>
+  <gazebo reference="right_wheel">
+    <material>Gazebo/Red</material>
+  </gazebo>
   <joint type="continuous" name="left_wheel_hinge">
-    <origin xyz="0 0.15 0" rpy="0 0 0"/>
-    <child link="left_wheel"/>
-    <parent link="chassis"/>
-    <axis xyz="0 1 0" rpy="0 0 0"/>
-    <limit effort="10000" velocity="1000"/>
-    <dynamics damping="1.0" friction="1.0"/>
+    <origin xyz="0 0.325 0" rpy="0 0 0" />
+    <child link="left_wheel" />
+    <parent link="chassis" />
+    <axis xyz="0 1 0" rpy="0 0 0" />
+    <limit effort="10000" velocity="1000" />
+    <dynamics damping="1.0" friction="1.0" />
   </joint>
   <joint type="continuous" name="right_wheel_hinge">
-    <origin xyz="0 -0.15 0" rpy="0 0 0"/>
-    <child link="right_wheel"/>
-    <parent link="chassis"/>
-    <axis xyz="0 1 0" rpy="0 0 0"/>
-    <limit effort="10000" velocity="1000"/>
-    <dynamics damping="1.0" friction="1.0"/>
+    <origin xyz="0 -0.325 0" rpy="0 0 0" />
+    <child link="right_wheel" />
+    <parent link="chassis" />
+    <axis xyz="0 1 0" rpy="0 0 0" />
+    <limit effort="10000" velocity="1000" />
+    <dynamics damping="1.0" friction="1.0" />
   </joint>
-  <link name='camera'>
-    <pose>0 0 0 0 0 0</pose>
-    <inertial>
-      <mass value="0.1"/>
-      <origin xyz="0.0 0 0" rpy="0.0 0 0"/>
-      <inertia
-          ixx="1e-6" ixy="0" ixz="0"
-          iyy="1e-6" iyz="0"
-          izz="1e-6"
-      />
-    </inertial>
-    <collision name='collision'>
-      <origin xyz="0 0 0" rpy=" 0 0 0"/>
+  <link name="camera">
+    <box_inertia x="0.05" y="0.05" z="0.05" m="0.1" />
+    <collision>
+      <origin xyz="0 0 0" rpy="0 0 0" />
       <geometry>
-        <box size="0.05 0.05 0.05"/>
+        <box size="0.05 0.05 0.05" />
       </geometry>
     </collision>
-    <visual name='camera_visual'>
-      <origin xyz="0 0 0" rpy="0 0 0"/>
+    <visual>
+      <origin xyz="0 0 0" rpy="0 0 0" />
       <geometry>
-        <box size="0.05 0.05 0.05"/>
+        <box size="0.05 0.05 0.05" />
       </geometry>
     </visual>
   </link>
+  <gazebo reference="camera">
+    <material>Gazebo/Green</material>
+  </gazebo>
   <joint type="fixed" name="camera_joint">
-    <origin xyz="0.2 0 0" rpy="0 0 0"/>
-    <child link="camera"/>
-    <parent link="chassis"/>
-    <axis xyz="0 1 0" rpy="0 0 0"/>
-    <limit effort="10000" velocity="1000"/>
-    <dynamics damping="1.0" friction="1.0"/>
+    <origin xyz="0.3 0 0" rpy="0 0 0" />
+    <parent link="chassis" />
+    <child link="camera" />
   </joint>
-  <link name='hokuyo'>
-    <pose>0 0 0 0 0 0</pose>
+  <link name="hokuyo">
     <inertial>
-      <mass value="1e-5"/>
-      <origin xyz="0.0 0 0" rpy="0.0 0 0"/>
+      <mass value="1e-5" />
       <inertia
-          ixx="1e-6" ixy="0" ixz="0"
-          iyy="1e-6" iyz="0"
-          izz="1e-6"
+        ixx="1e-6" ixy="0" ixz="0"
+        iyy="1e-6" iyz="0"
+        izz="1e-6"
       />
     </inertial>
-    <collision name='collision'>
-      <origin xyz="0 0 0" rpy=" 0 0 0"/>
+    <collision>
+      <origin xyz="0 0 0" rpy="0 0 0" />
       <geometry>
-        <box size="0.1 0.1 0.1"/>
+        <box size="0.1 0.1 0.1" />
       </geometry>
     </collision>
-    <visual name='hokuyo_visual'>
-      <origin xyz="0 0 0" rpy="0 0 0"/>
+    <visual>
+      <origin xyz="0 0 0" rpy="0 0 0" />
       <geometry>
-        <mesh filename="package://my_robot/meshes/hokuyo.dae"/>
+        <mesh filename="package://my_robot/meshes/hokuyo.dae" />
       </geometry>
     </visual>
   </link>
-  <joint type="fixed" name="hokuyo_joint">
-    <origin xyz="0.15 0.0 0.1" rpy="0 0 0"/>
-    <child link="hokuyo"/>
-    <parent link="chassis"/>
-    <axis xyz="0 1 0" rpy="0 0 0"/>
-    <limit effort="10000" velocity="1000"/>
-    <dynamics damping="1.0" friction="1.0"/>
+  <joint name="hokuyo" type="fixed">
+    <origin xyz="0.25 0 0.08" rpy="0 0 0"/>
+    <parent link="chassis" />
+    <child link="hokuyo" />
   </joint>
 </robot>

Commit message: update my_robot.xacro

File: my_robot/urdf/my_robot.xacro (robot description, xacro)
@@ -115,5 +115,5 @@
   </link>
   <gazebo reference="left_wheel">
-    <material>Gazebo/Blue</material>
+    <material>Gazebo/Red</material>
   </gazebo>
   <gazebo reference="right_wheel">
